File: hardware/kicad/pc070_aida_hdmi_dp/pc070_aida_hdmi_dp.kicad_pcb (KiCad board)
At the start: 4 copper layers, 40 x 150 mm, 16 parts, among them J1 47272-0001, J10 HDMR-19-01-S-SM-TR, J11 47272-0001, J12 HDMR-19-01-S-SM-TR, J2 HDMR-19-01-S-SM-TR, J3 47272-0001, J4 HDMR-19-01-S-SM-TR, J5 47272-0001, J6 HDMR-19-01-S-SM-TR, J7 47272-0001, J8 HDMR-19-01-S-SM-TR, J9 47272-0001

Commit message: Minor tidying of artwork
Parts:
- H1, H2, H3, H4: footprint MountingHole:MountingHole_5.3mm_M5_ISO7380_Pad_TopBottom -> MountingHole:MountingHole_3.2mm_M3_DIN965_Pad_TopBottom

Commit message: Producing artwork for bug-fixed bodge board
Connections:
- J1 pad 1: /pc070_aida_hdmi_dp_single/CLK -> /pc070_aida_hdmi_dp_single/SPARE*
- J1 pad 10: /pc070_aida_hdmi_dp_single/SPARE -> /pc070_aida_hdmi_dp_single/CLK*
- J1 pad 12: /pc070_aida_hdmi_dp_single/SPARE* -> /pc070_aida_hdmi_dp_single/CLK
- J1 pad 3: /pc070_aida_hdmi_dp_single/CLK* -> /pc070_aida_hdmi_dp_single/SPARE
- J1 pad 4: /pc070_aida_hdmi_dp_single/CONT -> /pc070_aida_hdmi_dp_single/BUSY*
- J1 pad 6: /pc070_aida_hdmi_dp_single/CONT* -> /pc070_aida_hdmi_dp_single/BUSY
- J1 pad 7: /pc070_aida_hdmi_dp_single/BUSY -> /pc070_aida_hdmi_dp_single/CONT*
- J1 pad 9: /pc070_aida_hdmi_dp_single/BUSY* -> /pc070_aida_hdmi_dp_single/CONT
- J11 pad 1: /pc070_aida_hdmi_dp_single3/CLK -> /pc070_aida_hdmi_dp_single3/SPARE*
- J11 pad 10: /pc070_aida_hdmi_dp_single3/SPARE -> /pc070_aida_hdmi_dp_single3/CLK*
- J11 pad 12: /pc070_aida_hdmi_dp_single3/SPARE* -> /pc070_aida_hdmi_dp_single3/CLK
- J11 pad 3: /pc070_aida_hdmi_dp_single3/CLK* -> /pc070_aida_hdmi_dp_single3/SPARE
- J11 pad 4: /pc070_aida_hdmi_dp_single3/CONT -> /pc070_aida_hdmi_dp_single3/BUSY*
- J11 pad 6: /pc070_aida_hdmi_dp_single3/CONT* -> /pc070_aida_hdmi_dp_single3/BUSY
- J11 pad 7: /pc070_aida_hdmi_dp_single3/BUSY -> /pc070_aida_hdmi_dp_single3/CONT*
- J11 pad 9: /pc070_aida_hdmi_dp_single3/BUSY* -> /pc070_aida_hdmi_dp_single3/CONT
- J3 pad 1: /pc070_aida_hdmi_dp_single1/CLK -> /pc070_aida_hdmi_dp_single1/SPARE*
- J3 pad 10: /pc070_aida_hdmi_dp_single1/SPARE -> /pc070_aida_hdmi_dp_single1/CLK*
- J3 pad 12: /pc070_aida_hdmi_dp_single1/SPARE* -> /pc070_aida_hdmi_dp_single1/CLK
- J3 pad 3: /pc070_aida_hdmi_dp_single1/CLK* -> /pc070_aida_hdmi_dp_single1/SPARE
- J3 pad 4: /pc070_aida_hdmi_dp_single1/CONT -> /pc070_aida_hdmi_dp_single1/BUSY*
- J3 pad 6: /pc070_aida_hdmi_dp_single1/CONT* -> /pc070_aida_hdmi_dp_single1/BUSY
- J3 pad 7: /pc070_aida_hdmi_dp_single1/BUSY -> /pc070_aida_hdmi_dp_single1/CONT*
- J3 pad 9: /pc070_aida_hdmi_dp_single1/BUSY* -> /pc070_aida_hdmi_dp_single1/CONT
- J5 pad 1: /pc070_aida_hdmi_dp_single2/CLK -> /pc070_aida_hdmi_dp_single2/SPARE*
- J5 pad 10: /pc070_aida_hdmi_dp_single2/SPARE -> /pc070_aida_hdmi_dp_single2/CLK*
- J5 pad 12: /pc070_aida_hdmi_dp_single2/SPARE* -> /pc070_aida_hdmi_dp_single2/CLK
- J5 pad 3: /pc070_aida_hdmi_dp_single2/CLK* -> /pc070_aida_hdmi_dp_single2/SPARE
- J5 pad 4: /pc070_aida_hdmi_dp_single2/CONT -> /pc070_aida_hdmi_dp_single2/BUSY*
- J5 pad 6: /pc070_aida_hdmi_dp_single2/CONT* -> /pc070_aida_hdmi_dp_single2/BUSY
- J5 pad 7: /pc070_aida_hdmi_dp_single2/BUSY -> /pc070_aida_hdmi_dp_single2/CONT*
- J5 pad 9: /pc070_aida_hdmi_dp_single2/BUSY* -> /pc070_aida_hdmi_dp_single2/CONT
- J7 pad 1: /pc070_aida_hdmi_dp_single5/CLK -> /pc070_aida_hdmi_dp_single5/SPARE*
- J7 pad 10: /pc070_aida_hdmi_dp_single5/SPARE -> /pc070_aida_hdmi_dp_single5/CLK*
- J7 pad 12: /pc070_aida_hdmi_dp_single5/SPARE* -> /pc070_aida_hdmi_dp_single5/CLK
- J7 pad 3: /pc070_aida_hdmi_dp_single5/CLK* -> /pc070_aida_hdmi_dp_single5/SPARE
- J7 pad 4: /pc070_aida_hdmi_dp_single5/CONT -> /pc070_aida_hdmi_dp_single5/BUSY*
- J7 pad 6: /pc070_aida_hdmi_dp_single5/CONT* -> /pc070_aida_hdmi_dp_single5/BUSY
- J7 pad 7: /pc070_aida_hdmi_dp_single5/BUSY -> /pc070_aida_hdmi_dp_single5/CONT*
- J7 pad 9: /pc070_aida_hdmi_dp_single5/BUSY* -> /pc070_aida_hdmi_dp_single5/CONT
- J9 pad 1: /pc070_aida_hdmi_dp_single4/CLK -> /pc070_aida_hdmi_dp_single4/SPARE*
- J9 pad 10: /pc070_aida_hdmi_dp_single4/SPARE -> /pc070_aida_hdmi_dp_single4/CLK*
- J9 pad 12: /pc070_aida_hdmi_dp_single4/SPARE* -> /pc070_aida_hdmi_dp_single4/CLK
- J9 pad 3: /pc070_aida_hdmi_dp_single4/CLK* -> /pc070_aida_hdmi_dp_single4/SPARE
- J9 pad 4: /pc070_aida_hdmi_dp_single4/CONT -> /pc070_aida_hdmi_dp_single4/BUSY*
- J9 pad 6: /pc070_aida_hdmi_dp_single4/CONT* -> /pc070_aida_hdmi_dp_single4/BUSY
- J9 pad 7: /pc070_aida_hdmi_dp_single4/BUSY -> /pc070_aida_hdmi_dp_single4/CONT*
- J9 pad 9: /pc070_aida_hdmi_dp_single4/BUSY* -> /pc070_aida_hdmi_dp_single4/CONT
Routing:
- net /pc070_aida_hdmi_dp_single3/TRIG*: track 25.6 -> 41.1 mm, vias 2 -> 0
- net /pc070_aida_hdmi_dp_single/TRIG*: track 25.6 -> 41.1 mm, vias 2 -> 0
- net /pc070_aida_hdmi_dp_single4/TRIG*: track 25.6 -> 41.1 mm, vias 2 -> 0
- net /pc070_aida_hdmi_dp_single2/TRIG*: track 25.6 -> 41.1 mm, vias 2 -> 0
- net /pc070_aida_hdmi_dp_single5/TRIG*: track 25.6 -> 41.1 mm, vias 2 -> 0
- net /pc070_aida_hdmi_dp_single1/TRIG*: track 25.6 -> 41.1 mm, vias 2 -> 0
- net /pc070_aida_hdmi_dp_single3/TRIG: track 26.4 -> 41.1 mm, vias 2 -> 0
- net /pc070_aida_hdmi_dp_single1/TRIG: track 26.4 -> 41.1 mm, vias 2 -> 0
- net /pc070_aida_hdmi_dp_single4/TRIG: track 26.4 -> 41.1 mm, vias 2 -> 0
- net /pc070_aida_hdmi_dp_single/TRIG: track 26.4 -> 41.1 mm, vias 2 -> 0
- net /pc070_aida_hdmi_dp_single5/TRIG: track 26.4 -> 41.1 mm, vias 2 -> 0
- net /pc070_aida_hdmi_dp_single2/TRIG: track 26.4 -> 41.1 mm, vias 2 -> 0
- net /pc070_aida_hdmi_dp_single2/CLK: track 26.4 -> 18.3 mm, vias 2 -> 0
- net /pc070_aida_hdmi_dp_single1/CLK: track 26.4 -> 18.3 mm, vias 2 -> 0
- net /pc070_aida_hdmi_dp_single/CLK: track 26.4 -> 18.3 mm, vias 2 -> 0
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- added copper zone on B.Cu, net GND
- removed copper zone on In1.Cu, net GND
- removed copper zone on In2.Cu, net GND
Other:
- copper layers 4 -> 2
- board text added: "pc070_aida_hdmi v2 30 Sept 22 D. Cussans"

Commit message: Committing artwork for v3 of the adaptor board
Parts:
- added TP1: TestPoint, TestPoint:TestPoint_THTPad_1.0x1.0mm_Drill0.5mm, F.Cu at (91.1, 52.1)
- added TP10: TestPoint, TestPoint:TestPoint_THTPad_1.0x1.0mm_Drill0.5mm, F.Cu at (92.1, 57.9)
- added TP11: TestPoint, TestPoint:TestPoint_THTPad_1.0x1.0mm_Drill0.5mm, F.Cu at (92.1, 62.9)
- added TP12: TestPoint, TestPoint:TestPoint_THTPad_1.0x1.0mm_Drill0.5mm, F.Cu at (94.1, 62.9)
- added TP13: TestPoint, TestPoint:TestPoint_THTPad_1.0x1.0mm_Drill0.5mm, F.Cu at (91.1, 74.8)
- added TP14: TestPoint, TestPoint:TestPoint_THTPad_1.0x1.0mm_Drill0.5mm, F.Cu at (88.8, 88.3)
- added TP15: TestPoint, TestPoint:TestPoint_THTPad_1.0x1.0mm_Drill0.5mm, F.Cu at (87.8, 78.0)
- added TP16: TestPoint, TestPoint:TestPoint_THTPad_1.0x1.0mm_Drill0.5mm, F.Cu at (89.8, 78.0)
- added TP17: TestPoint, TestPoint:TestPoint_THTPad_1.0x1.0mm_Drill0.5mm, F.Cu at (88.8, 90.8)
- added TP18: TestPoint, TestPoint:TestPoint_THTPad_1.0x1.0mm_Drill0.5mm, F.Cu at (88.8, 92.8)
- added TP19: TestPoint, TestPoint:TestPoint_THTPad_1.0x1.0mm_Drill0.5mm, F.Cu at (92.1, 83.0)
- added TP2: TestPoint, TestPoint:TestPoint_THTPad_1.0x1.0mm_Drill0.5mm, F.Cu at (88.8, 65.7)
- added TP20: TestPoint, TestPoint:TestPoint_THTPad_1.0x1.0mm_Drill0.5mm, F.Cu at (94.1, 83.0)
- added TP21: TestPoint, TestPoint:TestPoint_THTPad_1.0x1.0mm_Drill0.5mm, F.Cu at (90.1, 80.5)
- added TP22: TestPoint, TestPoint:TestPoint_THTPad_1.0x1.0mm_Drill0.5mm, F.Cu at (92.1, 80.5)
- added TP23: TestPoint, TestPoint:TestPoint_THTPad_1.0x1.0mm_Drill0.5mm, F.Cu at (92.1, 85.5)
- added TP24: TestPoint, TestPoint:TestPoint_THTPad_1.0x1.0mm_Drill0.5mm, F.Cu at (94.1, 85.5)
- added TP25: TestPoint, TestPoint:TestPoint_THTPad_1.0x1.0mm_Drill0.5mm, F.Cu at (91.1, 97.4)
- added TP26: TestPoint, TestPoint:TestPoint_THTPad_1.0x1.0mm_Drill0.5mm, F.Cu at (88.8, 110.9)
- added TP27: TestPoint, TestPoint:TestPoint_THTPad_1.0x1.0mm_Drill0.5mm, F.Cu at (87.8, 100.6)
- added TP28: TestPoint, TestPoint:TestPoint_THTPad_1.0x1.0mm_Drill0.5mm, F.Cu at (89.8, 100.6)
- added TP29: TestPoint, TestPoint:TestPoint_THTPad_1.0x1.0mm_Drill0.5mm, F.Cu at (88.8, 113.4)
- added TP3: TestPoint, TestPoint:TestPoint_THTPad_1.0x1.0mm_Drill0.5mm, F.Cu at (87.8, 55.4)
- added TP30: TestPoint, TestPoint:TestPoint_THTPad_1.0x1.0mm_Drill0.5mm, F.Cu at (88.8, 115.4)
- added TP31: TestPoint, TestPoint:TestPoint_THTPad_1.0x1.0mm_Drill0.5mm, F.Cu at (92.1, 105.6)
- added TP32: TestPoint, TestPoint:TestPoint_THTPad_1.0x1.0mm_Drill0.5mm, F.Cu at (94.1, 105.6)
- added TP33: TestPoint, TestPoint:TestPoint_THTPad_1.0x1.0mm_Drill0.5mm, F.Cu at (90.1, 103.1)
- added TP34: TestPoint, TestPoint:TestPoint_THTPad_1.0x1.0mm_Drill0.5mm, F.Cu at (92.1, 103.1)
- added TP35: TestPoint, TestPoint:TestPoint_THTPad_1.0x1.0mm_Drill0.5mm, F.Cu at (92.1, 108.1)
- added TP36: TestPoint, TestPoint:TestPoint_THTPad_1.0x1.0mm_Drill0.5mm, F.Cu at (94.1, 108.1)
- added TP37: TestPoint, TestPoint:TestPoint_THTPad_1.0x1.0mm_Drill0.5mm, F.Cu at (91.1, 120.0)
- added TP38: TestPoint, TestPoint:TestPoint_THTPad_1.0x1.0mm_Drill0.5mm, F.Cu at (88.8, 133.5)
- added TP39: TestPoint, TestPoint:TestPoint_THTPad_1.0x1.0mm_Drill0.5mm, F.Cu at (87.8, 123.2)
- added TP4: TestPoint, TestPoint:TestPoint_THTPad_1.0x1.0mm_Drill0.5mm, F.Cu at (89.8, 55.4)
- added TP40: TestPoint, TestPoint:TestPoint_THTPad_1.0x1.0mm_Drill0.5mm, F.Cu at (89.8, 123.2)
- added TP41: TestPoint, TestPoint:TestPoint_THTPad_1.0x1.0mm_Drill0.5mm, F.Cu at (88.8, 136.0)
- added TP42: TestPoint, TestPoint:TestPoint_THTPad_1.0x1.0mm_Drill0.5mm, F.Cu at (88.8, 138.0)
- added TP43: TestPoint, TestPoint:TestPoint_THTPad_1.0x1.0mm_Drill0.5mm, F.Cu at (92.1, 128.2)
- added TP44: TestPoint, TestPoint:TestPoint_THTPad_1.0x1.0mm_Drill0.5mm, F.Cu at (94.1, 128.2)
- added TP45: TestPoint, TestPoint:TestPoint_THTPad_1.0x1.0mm_Drill0.5mm, F.Cu at (90.1, 125.7)
- added TP46: TestPoint, TestPoint:TestPoint_THTPad_1.0x1.0mm_Drill0.5mm, F.Cu at (92.1, 125.7)
- added TP47: TestPoint, TestPoint:TestPoint_THTPad_1.0x1.0mm_Drill0.5mm, F.Cu at (92.1, 130.7)
- added TP48: TestPoint, TestPoint:TestPoint_THTPad_1.0x1.0mm_Drill0.5mm, F.Cu at (94.1, 130.7)
- added TP49: TestPoint, TestPoint:TestPoint_THTPad_1.0x1.0mm_Drill0.5mm, F.Cu at (91.1, 142.6)
- added TP5: TestPoint, TestPoint:TestPoint_THTPad_1.0x1.0mm_Drill0.5mm, F.Cu at (88.8, 68.2)
- added TP50: TestPoint, TestPoint:TestPoint_THTPad_1.0x1.0mm_Drill0.5mm, F.Cu at (88.8, 156.1)
- added TP51: TestPoint, TestPoint:TestPoint_THTPad_1.0x1.0mm_Drill0.5mm, F.Cu at (87.8, 145.8)
- added TP52: TestPoint, TestPoint:TestPoint_THTPad_1.0x1.0mm_Drill0.5mm, F.Cu at (89.8, 145.8)
- added TP53: TestPoint, TestPoint:TestPoint_THTPad_1.0x1.0mm_Drill0.5mm, F.Cu at (88.8, 158.6)
- added TP54: TestPoint, TestPoint:TestPoint_THTPad_1.0x1.0mm_Drill0.5mm, F.Cu at (88.8, 160.6)
- added TP55: TestPoint, TestPoint:TestPoint_THTPad_1.0x1.0mm_Drill0.5mm, F.Cu at (92.1, 150.8)
- added TP56: TestPoint, TestPoint:TestPoint_THTPad_1.0x1.0mm_Drill0.5mm, F.Cu at (94.1, 150.8)
- added TP57: TestPoint, TestPoint:TestPoint_THTPad_1.0x1.0mm_Drill0.5mm, F.Cu at (90.1, 148.3)
- added TP58: TestPoint, TestPoint:TestPoint_THTPad_1.0x1.0mm_Drill0.5mm, F.Cu at (92.1, 148.3)
- added TP59: TestPoint, TestPoint:TestPoint_THTPad_1.0x1.0mm_Drill0.5mm, F.Cu at (92.1, 153.3)
- added TP6: TestPoint, TestPoint:TestPoint_THTPad_1.0x1.0mm_Drill0.5mm, F.Cu at (88.8, 70.2)
- added TP60: TestPoint, TestPoint:TestPoint_THTPad_1.0x1.0mm_Drill0.5mm, F.Cu at (94.1, 153.3)
- added TP61: TestPoint, TestPoint:TestPoint_THTPad_1.0x1.0mm_Drill0.5mm, F.Cu at (91.1, 165.2)
- added TP62: TestPoint, TestPoint:TestPoint_THTPad_1.0x1.0mm_Drill0.5mm, F.Cu at (88.8, 178.7)
- added TP63: TestPoint, TestPoint:TestPoint_THTPad_1.0x1.0mm_Drill0.5mm, F.Cu at (87.8, 168.4)
- added TP64: TestPoint, TestPoint:TestPoint_THTPad_1.0x1.0mm_Drill0.5mm, F.Cu at (89.8, 168.4)
- added TP65: TestPoint, TestPoint:TestPoint_THTPad_1.0x1.0mm_Drill0.5mm, F.Cu at (88.8, 181.2)
- added TP66: TestPoint, TestPoint:TestPoint_THTPad_1.0x1.0mm_Drill0.5mm, F.Cu at (88.8, 183.2)
- added TP67: TestPoint, TestPoint:TestPoint_THTPad_1.0x1.0mm_Drill0.5mm, F.Cu at (92.1, 173.4)
- added TP68: TestPoint, TestPoint:TestPoint_THTPad_1.0x1.0mm_Drill0.5mm, F.Cu at (94.1, 173.4)
- added TP69: TestPoint, TestPoint:TestPoint_THTPad_1.0x1.0mm_Drill0.5mm, F.Cu at (90.1, 170.9)
- added TP7: TestPoint, TestPoint:TestPoint_THTPad_1.0x1.0mm_Drill0.5mm, F.Cu at (92.1, 60.4)
- added TP70: TestPoint, TestPoint:TestPoint_THTPad_1.0x1.0mm_Drill0.5mm, F.Cu at (92.1, 170.9)
- added TP71: TestPoint, TestPoint:TestPoint_THTPad_1.0x1.0mm_Drill0.5mm, F.Cu at (92.1, 175.9)
- added TP72: TestPoint, TestPoint:TestPoint_THTPad_1.0x1.0mm_Drill0.5mm, F.Cu at (94.1, 175.9)
- added TP8: TestPoint, TestPoint:TestPoint_THTPad_1.0x1.0mm_Drill0.5mm, F.Cu at (94.1, 60.4)
- added TP9: TestPoint, TestPoint:TestPoint_THTPad_1.0x1.0mm_Drill0.5mm, F.Cu at (90.1, 57.9)
Connections:
- J1 pad 16: /pc070_aida_hdmi_dp_single/TRIG* -> GND
- J1 pad 17: GND -> /pc070_aida_hdmi_dp_single/TRIG*
- J10 pad 16: GND -> /pc070_aida_hdmi_dp_single4/TRIG*
- J10 pad 17: /pc070_aida_hdmi_dp_single4/TRIG* -> unconnected-(J10-Pad17)
- J11 pad 16: /pc070_aida_hdmi_dp_single3/TRIG* -> GND
- J11 pad 17: GND -> /pc070_aida_hdmi_dp_single3/TRIG*
- J12 pad 16: GND -> /pc070_aida_hdmi_dp_single3/TRIG*
- J12 pad 17: /pc070_aida_hdmi_dp_single3/TRIG* -> unconnected-(J12-Pad17)
- J2 pad 16: GND -> /pc070_aida_hdmi_dp_single/TRIG*
- J2 pad 17: /pc070_aida_hdmi_dp_single/TRIG* -> unconnected-(J2-Pad17)
- J3 pad 16: /pc070_aida_hdmi_dp_single1/TRIG* -> GND
- J3 pad 17: GND -> /pc070_aida_hdmi_dp_single1/TRIG*
- J4 pad 16: GND -> /pc070_aida_hdmi_dp_single1/TRIG*
- J4 pad 17: /pc070_aida_hdmi_dp_single1/TRIG* -> unconnected-(J4-Pad17)
- J5 pad 16: /pc070_aida_hdmi_dp_single2/TRIG* -> GND
- J5 pad 17: GND -> /pc070_aida_hdmi_dp_single2/TRIG*
- J6 pad 16: GND -> /pc070_aida_hdmi_dp_single2/TRIG*
- J6 pad 17: /pc070_aida_hdmi_dp_single2/TRIG* -> unconnected-(J6-Pad17)
- J7 pad 16: /pc070_aida_hdmi_dp_single5/TRIG* -> GND
- J7 pad 17: GND -> /pc070_aida_hdmi_dp_single5/TRIG*
- J8 pad 16: GND -> /pc070_aida_hdmi_dp_single5/TRIG*
- J8 pad 17: /pc070_aida_hdmi_dp_single5/TRIG* -> unconnected-(J8-Pad17)
- J9 pad 16: /pc070_aida_hdmi_dp_single4/TRIG* -> GND
- J9 pad 17: GND -> /pc070_aida_hdmi_dp_single4/TRIG*
Routing:
- net GND: track 102.1 -> 93.3 mm, vias 60 -> 54
- net /pc070_aida_hdmi_dp_single4/TRIG*: track 41.1 -> 43.7 mm
- net /pc070_aida_hdmi_dp_single3/TRIG*: track 41.1 -> 43.7 mm
- net /pc070_aida_hdmi_dp_single1/TRIG*: track 41.1 -> 43.7 mm
- net /pc070_aida_hdmi_dp_single/TRIG*: track 41.1 -> 43.7 mm
- net /pc070_aida_hdmi_dp_single2/TRIG*: track 41.1 -> 43.7 mm
- net /pc070_aida_hdmi_dp_single5/TRIG*: track 41.1 -> 43.7 mm
- net /pc070_aida_hdmi_dp_single2/BUSY*: track 18.0 -> 19.1 mm
- net /pc070_aida_hdmi_dp_single/BUSY*: track 18.0 -> 19.1 mm
- net /pc070_aida_hdmi_dp_single1/BUSY*: track 18.0 -> 19.1 mm
- net /pc070_aida_hdmi_dp_single5/BUSY*: track 18.0 -> 19.1 mm
- net /pc070_aida_hdmi_dp_single4/BUSY*: track 18.0 -> 19.1 mm
- net /pc070_aida_hdmi_dp_single3/BUSY*: track 18.0 -> 19.1 mm
- net /pc070_aida_hdmi_dp_single2/SPARE*: track 18.0 -> 18.9 mm
- net /pc070_aida_hdmi_dp_single/SPARE*: track 18.0 -> 18.9 mm
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Other:
- board text added: "pc070_aida_hdmi v3 20 Oct 22 D. Cussans"
- board text removed: "pc070_aida_hdmi v2 30 Sept 22 D. Cussans"
